File: kicad/mod/mod.kicad_pcb (KiCad board)
At the start: 0 parts

Commit message: Meh
Parts:
- added C1: 1µF, Capacitor_SMD:C_0805_2012Metric, F.Cu at (139.7, 101.6)
- added C2: 100nF, Capacitor_SMD:C_0805_2012Metric, F.Cu at (130.8, 100.0)
- added C3: 1µF, Capacitor_SMD:C_0805_2012Metric, F.Cu at (146.0, 102.4)
- added J1: In, Connector_PinHeader_2.00mm:PinHeader_2x03_P2.00mm_Vertical, F.Cu at (128.0, 90.0)
- added J2: Out, Connector_PinHeader_2.00mm:PinHeader_2x03_P2.00mm_Vertical, F.Cu at (133.5, 90.0)
- added J3: Program Pins, Connector_PinHeader_2.54mm:PinHeader_1x03_P2.54mm_Vertical, F.Cu at (154.5, 97.8)
- added R1: 4K7, Capacitor_SMD:C_0805_2012Metric, F.Cu at (135.2, 101.6)
- added U1: AP7384-33SA, Package_TO_SOT_SMD:SOT-23, F.Cu at (126.4, 104.0)
- added U2: ATtiny402-SS, Package_SO:SOIC-8_3.9x4.9mm_P1.27mm, F.Cu at (158.6, 87.4)
Other:
- copper layers 0 -> 2
